File: MiniProjectBoardProject.kicad_pcb (KiCad board)
At the start: 2 copper layers, 33 parts, among them J1 Conn_01x33_Male, J2 Conn_01x33_Male, SW1 SW_Push, SW2 SW_Push, U1 STM32F051R8Tx, U2 LD3985M33R_SOT23

Commit message: Finished PCB, missing Gerber
Parts:
- added G***: LOGO, Graphic:graphic, F.Cu at (109.2, 96.5)
- added J4: Conn_01x04_Male, Connector_PinSocket_2.54mm:PinSocket_1x04_P2.54mm_Vertical, F.Cu at (104.6, 122.6)
- added J5: Conn_01x04_Male, Connector_PinSocket_2.54mm:PinSocket_1x04_P2.54mm_Vertical, F.Cu at (125.2, 63.5)
- added J7: Conn_02x08_Odd_Even, Connector_PinSocket_2.54mm:PinSocket_2x08_P2.54mm_Vertical, B.Cu at (102.8, 139.0)
- J1, J2: footprint Connector_PinSocket_2.00mm:PinSocket_1x33_P2.00mm_Vertical -> Connector_PinSocket_2.54mm:PinSocket_1x33_P2.54mm_Vertical
- moved C2 48.2 mm to (106.0, 127.5)
- moved C6 46.5 mm to (97.3, 127.6)
- moved C7 45.8 mm to (99.7, 127.6)
- moved C10 45.7 mm to (122.9, 115.3)
- moved C8 45.0 mm to (102.2, 127.5)
- moved C3 44.8 mm to (121.2, 130.1)
- moved U1 44.4 mm to (111.0, 97.0)
- moved C11 44.4 mm to (116.1, 123.7)
- moved C12 44.4 mm to (121.2, 123.7)
- moved C5 44.4 mm to (116.1, 130.0)
- moved D1 44.4 mm to (111.0, 130.0)
- moved D2 44.4 mm to (112.3, 70.4)
- moved D4 44.4 mm to (107.2, 70.4)
- moved R5 44.4 mm to (116.1, 112.3)
- moved SW1 44.4 mm to (103.4, 76.7)
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Connections:
- J1 pad 3: -BATT -> VBAT
Routing:
- net VSS: track 0.00 -> 129.7 mm, vias 0 -> 16
- net +5V: track 0.00 -> 121.9 mm
- net PC14: track 0.00 -> 121.6 mm
- net PC13: track 0.00 -> 114.5 mm, vias 0 -> 2
- net PC10: track 0.00 -> 86.3 mm
- net Net-(D2-Pad2): track 0.00 -> 85.8 mm, vias 0 -> 2
- net PC3: track 0.00 -> 83.5 mm
- net PC12: track 0.00 -> 82.6 mm
- net PC2: track 0.00 -> 81.0 mm
- net PC1: track 0.00 -> 80.4 mm
- net PC11: track 0.00 -> 78.0 mm, vias 0 -> 1
- net PC5: track 0.00 -> 73.5 mm
- net PC0: track 0.00 -> 71.9 mm, vias 0 -> 2
- net PC7: track 0.00 -> 69.8 mm, vias 0 -> 2
- net PC6: track 0.00 -> 69.7 mm
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- added copper zone on F.Cu, net VBAT
- added copper zone on B.Cu, net VSS
Other:
- board outline added: 58.4 x 88.9 mm
- rule trace_min: 0.2 -> 0.1
- board text added: "+3V"
- board text added: "+5V"
- board text added: "BOOT0"
- board text added: "ECE362 Final Project - Rev: 1 Designed by: Alan Gregorian"
- board text added: "GND"
- board text added: "GND GND +5V +5V"
- board text added: "NRST"
- board text added: "PA0"
- board text added: "PA1"
- board text added: "PA10"
- board text added: "PA11"
- board text added: "PA12"
- board text added: "PA13"
- board text added: "PA14"
- board text added: "PA15"
- board text added: "PA2"
- board text added: "PA3"
- board text added: "PA4"
- board text added: "PA5"
- board text added: "PA6"
- board text added: "PA7"
- board text added: "PA8"
- board text added: "PA9"
- board text added: "PB0"
- board text added: "PB1"
- board text added: "PB10"
- board text added: "PB11"
- board text added: "PB12"
- board text added: "PB13"
- board text added: "PB14"
- board text added: "PB15"
- board text added: "PB2"
- board text added: "PB3"
- board text added: "PB4"
- board text added: "PB5"
- board text added: "PB6"
- board text added: "PB7"
- board text added: "PB8"
- board text added: "PB9"
- board text added: "PC0"
- board text added: "PC0 PC2 PC3 PC5 PC6 PC10 PC13 PC12"
- board text added: "PC1"
- board text added: "PC1 GND PC4 GND PC7 PC11 PC14 GND"
- board text added: "PC10"
- board text added: "PC11"
- board text added: "PC12"
- board text added: "PC13"
- board text added: "PC14"
- board text added: "PC15"
- board text added: "PC2"
- board text added: "PC3"
- board text added: "PC4"
- board text added: "PC5"
- board text added: "PC6"
- board text added: "PC7"
- board text added: "PC8"
- board text added: "PC9"
- board text added: "PD2"
- board text added: "PF0"
- board text added: "PF1"
- board text added: "PF4"
- board text added: "PF5"
- board text added: "PF6"
- board text added: "PF7"
- board text added: "RESET"
- board text added: "USER"
