File: MiniProjectBoardProject.sch (KiCad schematic (older format))
At the start: 32 parts, among them J1 Conn_01x33_Male, J2 Conn_01x33_Male, J3 Conn_02x08_Top_Bottom, J4 Conn_01x04_Male, J5 Conn_01x04_Male, SW1 SW_Push, SW2 SW_Push, U1 STM32F051R8Tx, U2 LD3985M33R_SOT23

Commit message: Finished PCB, missing Gerber
Parts:
- removed J3: Conn_02x08_Top_Bottom, Connector_PinSocket_2.54mm:PinSocket_2x08_P2.54mm_Vertical, symbol Connector_Generic:Conn_02x08_Top_Bottom
- added J7: Conn_02x08_Odd_Even, Connector_PinSocket_2.54mm:PinSocket_2x08_P2.54mm_Vertical, symbol Connector_Generic:Conn_02x08_Odd_Even
Connections:
- net -BATT is gone; now on net +3V3: J1.3 (Pin_3)
- net +3V3: no longer J4.1 (Pin_1), J4.2 (Pin_2)
- net +5V: now also J4.1 (Pin_1), J4.2 (Pin_2)
- net GNDREF: now also J7.16 (Pin_16), J7.4 (Pin_4), J7.8 (Pin_8)
- net PC0: now also J7.1 (Pin_1)
- net PC1: now also J7.2 (Pin_2)
- net PC10: now also J7.11 (Pin_11)
- net PC11: now also J7.12 (Pin_12)
- net PC12: now also J7.15 (Pin_15)
- net PC13: now also J7.13 (Pin_13)
- net PC14: now also J7.14 (Pin_14)
- net PC2: now also J7.3 (Pin_3)
- net PC3: now also J7.5 (Pin_5)
- net PC4: now also J7.6 (Pin_6)
- net PC5: now also J7.7 (Pin_7)
- net PC6: now also J7.9 (Pin_9)
- net PC7: now also J7.10 (Pin_10)
Other:
- note added: "BATTERY CONN."
- note added: "CAPACITIVE TOUCH CONN."
- note added: "GND CONN."
- note added: "POWER CONNECTION"
- moved on the sheet: D4, R3, R4
